File: kicad/ESP32.kicad_sch (KiCad schematic)
At the start: 45 parts, among them J501 GCT_MEM2075-00-140-01-A_DP, J502 USB_B_Micro, J503 Conn_02x05, U13 SN74LVC8T245DBR, U15 SN74LVC8T245DBR, U5 ESP32-S3-DevKitC, U501 SN74LVC1G125DBVR, U503 SN74LVC1G125DBVR, U508 SN74LVC1G125DBVR, U509 SN74LVC1G125DBVR

Commit message: Initial Release
Parts:
- J503: value Conn_02x05 -> Conn_02x05_Right_Angle; Digi-Key_PN 612-TSW-105-20-G-D-ND -> 2057-PH2RA-10-UA-ND; Digikey 612-TSW-105-20-G-D-ND -> 2057-PH2RA-10-UA-ND; MPN TSW-105-20-G-D -> PH2RA-10-UA; Manufacturer Samtec Inc. -> Adam Tech
Other:
- note added: "PROGRAMMING PORT"
Changed lines of the file:
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@@
     (effects (font (size 2.9972 2.9972) (thickness 0.5994) bold) (justify left bottom))
   )
+  (text "PROGRAMMING PORT" (at 137.16 81.28 0)
+    (effects (font (size 2.9972 2.9972) (thickness 0.5994) bold) (justify left bottom))
+  )
   (text "BLUE" (at 147.32 122.555 0)
     (effects (font (size 1.27 1.27)) (justify left bottom))
@@
       (effects (font (size 1.27 1.27)))
     )
-    (property "Value" "Conn_02x05" (at 240.03 164.4396 0)
+    (property "Value" "Conn_02x05_Right_Angle" (at 240.03 164.4396 0)
       (effects (font (size 1.27 1.27)) hide)
     )
@@
       (effects (font (size 1.27 1.27)) hide)
     )
-    (property "Datasheet" "https://suddendocs.samtec.com/catalog_english/tsw_th.pdf" (at 238.76 172.72 0)
+    (property "Datasheet" "https://app.adam-tech.com/products/download/data_sheet/200508/ph2ra-xx-ua-data-sheet.pdf" (at 238.76 172.72 0)
       (effects (font (size 1.27 1.27)) hide)
     )
-    (property "Description" "CONN HEADER VERT 10POS 2.54MM" (at 238.76 172.72 0)
+    (property "Description" "CONN HEADER R/A 10POS 2.54MM" (at 238.76 172.72 0)
       (effects (font (size 1.27 1.27)) hide)
     )
-    (property "Digi-Key_PN" "612-TSW-105-20-G-D-ND" (at 238.76 172.72 0)
+    (property "Digi-Key_PN" "2057-PH2RA-10-UA-ND" (at 238.76 172.72 0)
       (effects (font (size 1.27 1.27)) hide)
     )
-    (property "MPN" "TSW-105-20-G-D" (at 238.76 172.72 0)
+    (property "MPN" "PH2RA-10-UA" (at 238.76 172.72 0)
       (effects (font (size 1.27 1.27)) hide)
     )
-    (property "Manufacturer" "Samtec Inc." (at 238.76 172.72 0)
+    (property "Manufacturer" "Adam Tech" (at 238.76 172.72 0)
       (effects (font (size 1.27 1.27)) hide)
     )
-    (property "Digikey" "612-TSW-105-20-G-D-ND" (at 238.76 172.72 0)
+    (property "Digikey" "2057-PH2RA-10-UA-ND" (at 238.76 172.72 0)
       (effects (font (size 1.27 1.27)) hide)
     )
