File: kicad/RS232.kicad_sch (KiCad schematic)
At the start: 11 parts, among them J10 Conn_02x03, J11 Conn_02x03, J401 DB9_Male_MountingHoles, J403 DB9_Male_MountingHoles, U4 ICL3232CPZ

Commit message: Initial Release
Changed lines of the file:
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@@
     (stroke (width 0) (type default))
+  )
+  (text_box "Do not connect UART0_RX to a TX source as \nthe ESP32 USB-Serial IC is driving this signal."
+    (at 35.56 93.98 0) (size 50.8 5.08)
+    (stroke (width 0) (type default))
+    (fill (type none))
+    (effects (font (size 1.27 1.27)) (justify left top))
   )
   (text_box "RS232"
@@
     (effects (font (size 5.08 5.08) (thickness 1.016) bold) (justify left top))
   )
-  (text_box "If default jumpers are selected, external TTL \nlevel RS232 can be connected to pins 5 & 6 \n+ GND for ESP32 debug/download port connection.\n"
-    (at 33.02 157.48 0) (size 53.34 7.62)
-    (stroke (width 0) (type default))
-    (fill (type none))
-    (effects (font (size 1.27 1.27)) (justify left top))
-  )
-  (text_box "A place to add connection to external \nTTL level RS232 modules\n"
+  (text_box "A place to add connection to external \nTTL level RS232 modules.\n"
     (at 35.56 86.36 0) (size 43.18 5.08)
     (stroke (width 0) (type default))
@@
     (effects (font (size 1.27 1.27)) (justify left top))
   )
-  (text_box "J401 RS232 Output Options\nTo select ESP32 Console add jumpers\n1-3, 2-4\nTo select ESP32 Debug messages add jumpers\n3-5, 4-6\nDefault jumper settings\n1-3, 2-4\n"
+  (text_box "J401 RS232 Output Options\nTo select ESP32 Console add jumpers\n3-5, 4-6 (Uart 1 selected)\nTo select ESP32 Debug messages add jumper\n1-3      (Uart 0 selected)\nDefault jumper settings = Console\n3-5, 4-6 (Uart 1)\n"
     (at 33.02 134.62 0) (size 48.26 17.78)
     (stroke (width 0) (type default))
@@
     (effects (font (size 1.27 1.27)) (justify left top))
   )
-  (text_box "ESP32 Debug / Download option on uart 1 set in SW.\n"
-    (at 33.02 170.18 0) (size 53.34 5.08)
+  (text_box "ESP32 Console / Download option on uart 1 set in SW.\n"
+    (at 33.02 154.94 0) (size 58.42 5.08)
     (stroke (width 0) (type default))
     (fill (type none))
